File: Dock/Smart-Watch-L15-Dock.kicad_pcb (KiCad board)
At the start: 2 copper layers, 8.7 x 4.4 mm, 7 parts, among them J1 USB4125-GF-A, J2 Conn_01x06, U1 USBLC6-4SC6

Commit message: Watch Finalization and PCB Draft for the Dock
Parts:
- added G***: LOGO, LOGO, F.Cu at (107.0, 73.8)
- added P2: JTAG, 1_I_Syst.inc:CON10_2X5_DUK_FTSH_SAI-M, B.Cu at (98.1, 62.6)
- D1, J1, R1, R2, R3, U1: moved to B.Cu
- moved D1 77.1 mm to (103.8, 49.8), turned to 180 degrees
- moved R3 73.5 mm to (103.8, 52.0)
- moved U1 64.2 mm to (109.7, 59.0), turned to 180 degrees
- moved R2 57.5 mm to (97.2, 86.4), turned to 90 degrees
- moved J1 52.6 mm to (103.7, 88.2), turned to 180 degrees
- moved J2 49.8 mm to (98.4, 81.5), turned to 90 degrees
- moved R1 44.3 mm to (110.2, 86.4), turned to 90 degrees
Routing:
- net /nRESET: track 0.00 -> 62.2 mm, vias 0 -> 3
- net +5V: track 0.00 -> 49.1 mm
- net VDD: track 0.00 -> 49.1 mm, vias 0 -> 3
- net /SWDCLK: track 0.00 -> 40.1 mm, vias 0 -> 2
- net /SWDIO: track 0.00 -> 37.2 mm, vias 0 -> 2
- net Net-(J1-CC2): track 0.00 -> 7.58 mm
- net Net-(J1-CC1): track 0.00 -> 7.58 mm
- net GND: track 0.00 -> 5.94 mm, vias 0 -> 4
- net Net-(D1-A): track 0.00 -> 2.25 mm
- added copper zone on B.Cu, net GND
- added copper zone on F.Cu, net GND
Other:
- board size 8.7 x 4.4 mm -> 22 x 45 mm
- board text added: "2026"
- board text added: "BLYSTWATCH"
- board text added: "DOCK"
- board text added: "Rev1"
