File: Dock/Smart-Watch-L15-Dock.kicad_sch (KiCad schematic)
At the start: 8 parts, among them J1 USB4125-GF-A, J2 Conn_01x06, P2 ARM JTAG/SWD, U1 USBLC6-4SC6

Commit message: Watch Finalization and PCB Draft for the Dock
Parts:
- P2: footprint 1_I-SYST_inc:CON10_2X5_DUK_FTSH_SAI-M -> 1_I_Syst.inc:CON10_2X5_DUK_FTSH_SAI-M
Other:
- moved on the sheet: P2
