File: Watch/power_management.kicad_sch (KiCad schematic)
At the start: 10 parts, among them J5 Conn_01x03, J6 DOCK_PADS, U5 NPM1304-QEAA-R7

Commit message: Screenshots
Other:
- note added: "Watch to Docker Connection"
- moved on the sheet: J6
Changed lines of the file:
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@@
 		)
 	)
+	(text "Watch to Docker Connection"
+		(exclude_from_sim no)
+		(at 216.408 101.092 0)
+		(effects
+			(font
+				(size 1.905 1.905)
+			)
+		)
+	)
 	(text "SWCLK"
 		(exclude_from_sim no)
-		(at 206.248 105.918 0)
+		(at 206.248 114.808 0)
 		(effects
 			(font
@@
 	(wire
 		(pts
-			(xy 203.2 111.76) (xy 213.36 111.76)
+			(xy 203.2 120.65) (xy 213.36 120.65)
 		)
 		(stroke
@@
 	(wire
 		(pts
-			(xy 213.36 101.6) (xy 203.2 101.6)
+			(xy 213.36 110.49) (xy 203.2 110.49)
 		)
 		(stroke
@@
 	(wire
 		(pts
-			(xy 203.2 114.3) (xy 222.25 114.3)
+			(xy 203.2 123.19) (xy 222.25 123.19)
 		)
 		(stroke
@@
 	(wire
 		(pts
-			(xy 213.36 99.06) (xy 213.36 101.6)
+			(xy 213.36 107.95) (xy 213.36 110.49)
 		)
 		(stroke
@@
 	(wire
 		(pts
-			(xy 203.2 109.22) (xy 222.25 109.22)
+			(xy 203.2 118.11) (xy 222.25 118.11)
 		)
 		(stroke
@@
 	(wire
 		(pts
-			(xy 203.2 106.68) (xy 222.25 106.68)
+			(xy 203.2 115.57) (xy 222.25 115.57)
 		)
 		(stroke
@@
 	(wire
 		(pts
-			(xy 203.2 104.14) (xy 222.25 104.14)
+			(xy 203.2 113.03) (xy 222.25 113.03)
 		)
 		(stroke
@@
 	(wire
 		(pts
-			(xy 213.36 111.76) (xy 213.36 118.11)
+			(xy 213.36 120.65) (xy 213.36 127)
 		)
 		(stroke
@@
 	)
 	(label "VBUS"
-		(at 222.25 114.3 180)
+		(at 222.25 123.19 180)
 		(effects
 			(font
@@
 	(hierarchical_label "SWDCLK"
 		(shape input)
-		(at 222.25 106.68 0)
+		(at 222.25 115.57 0)
 		(effects
 			(font
@@
 	(hierarchical_label "SWDIO"
 		(shape input)
-		(at 222.25 109.22 0)
+		(at 222.25 118.11 0)
 		(effects
 			(font
@@
 	(hierarchical_label "nRESET"
 		(shape input)
-		(at 222.25 104.14 0)
+		(at 222.25 113.03 0)
 		(effects
 			(font
@@
 	(symbol
 		(lib_id "power:Earth")
-		(at 213.36 118.11 0)
+		(at 213.36 127 0)
 		(mirror y)
 		(unit 1)
@@
 		(fields_autoplaced yes)
 		(property "Reference" "#PWR025"
-			(at 213.36 124.46 0)
+			(at 213.36 133.35 0)
 			(hide yes)
 			(show_name no)
@@
 		)
 		(property "Value" "GND"
-			(at 213.36 123.19 0)
+			(at 213.36 132.08 0)
 			(show_name no)
 			(do_not_autoplace no)
@@
 		)
 		(property "Footprint" ""
-			(at 213.36 118.11 0)
+			(at 213.36 127 0)
 			(hide yes)
 			(show_name no)
@@
 		)
 		(property "Datasheet" ""
-			(at 213.36 118.11 0)
+			(at 213.36 127 0)
 			(hide yes)
 			(show_name no)
@@
 		)
 		(property "Description" "Power symbol creates a global label with name \"Earth\""
-			(at 213.36 118.11 0)
+			(at 213.36 127 0)
 			(hide yes)
 			(show_name no)
@@
 	(symbol
 		(lib_id "Connector_Generic:Conn_01x06")
-		(at 198.12 109.22 180)
+		(at 198.12 118.11 180)
 		(unit 1)
 		(body_style 1)
@@
 		(dnp no)
 		(property "Reference" "J6"
-			(at 197.866 99.06 0)
+			(at 197.866 107.95 0)
 			(show_name no)
 			(do_not_autoplace no)
@@
 		)
 		(property "Value" "DOCK_PADS"
-			(at 201.93 117.348 0)
+			(at 201.93 126.238 0)
 			(show_name no)
 			(do_not_autoplace no)
@@
 		)
 		(property "Footprint" "1_I_Syst.inc:Dock_Pads_6Pin"
-			(at 198.12 109.22 0)
+			(at 198.12 118.11 0)
 			(hide yes)
 			(show_name no)
@@
 		)
 		(property "Datasheet" ""
-			(at 198.12 109.22 0)
+			(at 198.12 118.11 0)
 			(hide yes)
 			(show_name no)
@@
 		)
 		(property "Description" "Generic connector, single row, 01x06, script generated (kicad-library-utils/schlib/autogen/connector/)"
-			(at 198.12 109.22 0)
+			(at 198.12 118.11 0)
 			(hide yes)
 			(show_name no)
@@
 		)
 		(property "Availability" ""
-			(at 198.12 109.22 0)
+			(at 198.12 118.11 0)
 			(hide yes)
 			(show_name no)
@@
 		)
 		(property "Check_prices" ""
-			(at 198.12 109.22 0)
+			(at 198.12 118.11 0)
 			(hide yes)
 			(show_name no)
@@
 		)
 		(property "Description_1" ""
-			(at 198.12 109.22 0)
+			(at 198.12 118.11 0)
 			(hide yes)
 			(show_name no)
@@
 		)
 		(property "MF" ""
-			(at 198.12 109.22 0)
+			(at 198.12 118.11 0)
 			(hide yes)
 			(show_name no)
@@
 		)
 		(property "MP" ""
-			(at 198.12 109.22 0)
+			(at 198.12 118.11 0)
 			(hide yes)
 			(show_name no)
@@
 		)
 		(property "Package" ""
-			(at 198.12 109.22 0)
+			(at 198.12 118.11 0)
 			(hide yes)
 			(show_name no)
@@
 		)
 		(property "Price" ""
-			(at 198.12 109.22 0)
+			(at 198.12 118.11 0)
 			(hide yes)
 			(show_name no)
@@
 		)
 		(property "Purchase-URL" ""
-			(at 198.12 109.22 0)
+			(at 198.12 118.11 0)
 			(hide yes)
 			(show_name no)
@@
 		)
 		(property "SnapEDA_Link" ""
-			(at 198.12 109.22 0)
+			(at 198.12 118.11 0)
 			(hide yes)
 			(show_name no)
@@
 	(symbol
 		(lib_id "power:VDD")
-		(at 213.36 99.06 0)
+		(at 213.36 107.95 0)
 		(unit 1)
 		(body_style 1)
@@
 		(dnp no)
 		(property "Reference" "#PWR024"
-			(at 213.36 102.87 0)
+			(at 213.36 111.76 0)
 			(hide yes)
 			(show_name no)
@@
 		)
 		(property "Value" "VDD"
-			(at 213.36 95.504 0)
+			(at 213.36 104.394 0)
 			(show_name no)
 			(do_not_autoplace no)
@@
 		)
 		(property "Footprint" ""
-			(at 213.36 99.06 0)
+			(at 213.36 107.95 0)
 			(hide yes)
 			(show_name no)
@@
 		)
 		(property "Datasheet" ""
-			(at 213.36 99.06 0)
+			(at 213.36 107.95 0)
 			(hide yes)
 			(show_name no)
@@
 		)
 		(property "Description" "Power symbol creates a global label with name \"VDD\""
-			(at 213.36 99.06 0)
+			(at 213.36 107.95 0)
 			(hide yes)
 			(show_name no)
